Commit message: better inertias; camera+differential plugin added

File: urdf/edumip_my_robot.xacro (robot description, xacro)
@@ -7,4 +7,6 @@
  <xacro:property name="body_width" value="0.050" />
  <xacro:property name="body_length" value="0.035" />
+ <xacro:property name="camera_link" value="0.05" />
+ <!-- Size of square 'camera' box -->
  <material name="body">
   <color rgba="0 0 0.8 1"/>
@@ -30,5 +32,5 @@
     <origin xyz="0 0 -0.2"/>
     <mass value="1"/>
-    <inertia ixx="1" ixy="0" ixz="0" iyy="1" iyz="0" izz="0"/>
+    <inertia ixx="0.01" ixy="0" ixz="0" iyy="0.01" iyz="0" izz="0.01"/>
   </inertial>
  </link>
@@ -50,5 +52,5 @@
     <origin rpy="1.57075 0 0" xyz="0 ${-wheel_width} 0"/>
     <mass value="0.2"/>
-    <inertia ixx="0.2" ixy="0" ixz="0" iyy="0.2" iyz="0" izz="0.2"/>
+    <inertia ixx="0.01" ixy="0" ixz="0" iyy="0.01" iyz="0" izz="0.01"/>
   </inertial>
  </link>
@@ -70,7 +72,33 @@
     <origin rpy="1.57075 0 0" xyz="0 ${wheel_width} 0"/>
     <mass value="0.2"/>
-    <inertia ixx="0.2" ixy="0" ixz="0" iyy="0.2" iyz="0" izz="0.2"/>
+    <inertia ixx="0.01" ixy="0" ixz="0" iyy="0.01" iyz="0" izz="0.01"/>
   </inertial>
- </link>
+  </link>
+  <link name="camera_link">
+    <collision>
+      <origin xyz="0 0 ${body_height}" rpy="0 0 0"/>
+      <geometry>
+    <box size="${camera_link} ${camera_link} ${camera_link}"/>
+      </geometry>
+    </collision>
+    <visual>
+      <origin xyz="0 0 ${body_height}" rpy="0 0 0"/>
+      <geometry>
+    <box size="${camera_link} ${camera_link} ${camera_link}"/>
+      </geometry>
+      <material name="body"/>
+    </visual>
+    <inertial>
+      <mass value="1e-5" />
+      <origin xyz="0 0 ${body_height}" rpy="0 0 0"/>
+      <inertia ixx="1e-6" ixy="0" ixz="0" iyy="1e-6" iyz="0" izz="1e-6" />
+    </inertial>
+  </link>
+  <joint name="camera_joint" type="fixed">
+    <axis xyz="0 1 0"/>
+    <origin xyz="${camera_link} 0 ${body_height}"/>
+    <parent link="edumip_body"/>
+    <child link="camera_link"/>
+  </joint>
 <joint name="wheelL_joint" type="continuous">
  <parent link="edumip_body"/>
@@ -102,3 +130,63 @@
    <mu2>0.2</mu2>
  </gazebo>
+ <gazebo>
+ <plugin name="differential_drive_controller" filename="libgazebo_ros_diff_drive.so">
+   <legacyMode>false</legacyMode>
+   <rosDebugLevel>3</rosDebugLevel>
+   <alwaysOn>true</alwaysOn>
+   <updateRate>10</updateRate>
+   <leftJoint>wheelL_joint</leftJoint>
+   <rightJoint>wheelR_joint</rightJoint>
+   <wheelSeparation>${wheel_sep}</wheelSeparation>
+   <wheelDiameter>${wheel_radius*2.0}</wheelDiameter>
+   <torque>0.1</torque>
+   <commandTopic>/edumip/cmd</commandTopic>
+   <odometryTopic>/edumip/odom</odometryTopic>
+   <odometryFrame>world</odometryFrame>
+   <robotBaseFrame>edumip_body</robotBaseFrame>
+   <publishTf>1</publishTf>
+   <publishWheelTF>false</publishWheelTF>
+   <publishWheelJointState>true</publishWheelJointState>
+   <wheelAcceleration>0</wheelAcceleration>
+   <wheelTorque>0.1</wheelTorque>
+   <odometrySource>world</odometrySource>
+ </plugin>
+</gazebo>
+<gazebo reference="camera_link">
+ <sensor type="camera" name="camera1">
+   <update_rate>30.0</update_rate>
+   <camera name="head">
+     <horizontal_fov>1.3962634</horizontal_fov>
+     <image>
+       <width>800</width>
+       <height>800</height>
+       <format>R8G8B8</format>
+     </image>
+     <clip>
+       <near>0.02</near>
+       <far>300</far>
+     </clip>
+     <noise>
+       <type>gaussian</type>
+       <mean>0.0</mean>
+       <stddev>0.007</stddev>
+     </noise>
+   </camera>
+   <plugin name="camera_controller" filename="libgazebo_ros_camera.so">
+     <robotNamespace>edumip</robotNamespace>
+     <alwaysOn>true</alwaysOn>
+     <updateRate>10.0</updateRate>
+     <cameraName>camera1</cameraName>
+     <imageTopicName>image_raw</imageTopicName>
+     <cameraInfoTopicName>camera_info</cameraInfoTopicName>
+     <frameName>camera_link</frameName>
+     <hackBaseline>0.07</hackBaseline>
+     <distortionK1>0.0</distortionK1>
+     <distortionK2>0.0</distortionK2>
+     <distortionK3>0.0</distortionK3>
+     <distortionT1>0.0</distortionT1>
+     <distortionT2>0.0</distortionT2>
+   </plugin>
+ </sensor>
+</gazebo>
 </robot>
